File: ram_board.sch (KiCad schematic (older format))
At the start: 17 parts, among them J1 Bus, J2 PWR, U1 CPU - Z84C0010AEG, U2 IS61LV5128AL-10TLI, U3 SST39VF040-70-4C-NHE, U4 74LVC2G240, X1 ASV-xxxMHz

Commit message: re-gridded
Parts:
- removed C5: 100nF, Capacitor_SMD:C_0603_1608Metric_Pad1.05x0.95mm_HandSolder, symbol Device:C_Small
- X1: value ASV-xxxMHz -> ASV-20MHz
- renumbered C3 to C1, C1 to C2, C2 to C3, U2 to U1, U3 to U2, U1 to U3
Connections:
- net labels added: 1V8, 3V3, 5V
- net labels removed: +3.3V, +5V
- wire segments 177 -> 175
- no-connect marks 4 -> 0
Other:
- note removed: "red"
- moved on the sheet: C1, C2, C3, C4, D1, D2, J1, J2, R1, R2, R3, U1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

Commit message: Added plcc socket to library
Parts:
- removed U1: IS61LV5128AL-10TLI, Package_SO:TSOP-II-44_10.16x18.41mm_P0.8mm, symbol ram_board-rescue:IS61LV5128AL-10TLI-Memory_RAM
- added C5, C6: 100nF, Capacitor_SMD:C_0603_1608Metric_Pad1.05x0.95mm_HandSolder, symbol Device:C_Small
- added U1: IS61C5128AL-10TLI, Package_SO:TSOP-II-44_10.16x18.41mm_P0.8mm, symbol Memory_RAM:IS61C5128AL-10TLI
- U3: symbol sbc_z80-rescue:Z84C0010AEG -> ram_board-rescue:Z84C0010AEG-sbc_z80-rescue
- U4: renamed from U2; footprint Package_LCC:PLCC-32_SMD-Socket -> ram_rom_brd:PLCC-32_SMD-Socket
- renumbered U4 to U2
Connections:
- wire segments 175 -> 192
Other:
- moved on the sheet: C1, C2, C4, D2, R1, R2, R3
